Commit message: update vehicle_simulator

File: src/vehicle_simulator/urdf/rgbd_camera.urdf.xacro (robot description, xacro)
@@ -34,5 +34,5 @@
         </clip>
       </camera>
-      <plugin name="rgbd_camera_controller" filename="libgazebo_ros_depth_camera.so">
+      <plugin name="depth_camera_controller" filename="libgazebo_ros_camera.so">
         <alwaysOn>true</alwaysOn>
           <baseline>0.2</baseline>
@@ -42,5 +42,5 @@
           <depthImageTopicName>/rgbd_camera/depth/image</depthImageTopicName>
           <depthImageCameraInfoTopicName>/rgbd_camera/depth/camera_info</depthImageCameraInfoTopicName>
-          <pointCloudTopicName>/rgbd_camera/depth/points</pointCloudTopicName>
+          <pointCloudTopicName>/rgbd_camera/points</pointCloudTopicName>
           <frameName>rgbd_camera</frameName>
           <pointCloudCutoff>0.1</pointCloudCutoff>

File: src/vehicle_simulator/urdf/robot.urdf.xacro (robot description, xacro)
@@ -8,5 +8,13 @@
     <visual>
       <origin xyz="0 0 0" rpy="0 0 0"/>
+      <geometry>
+        <box size="0.01 0.01 0.01"/>
+      </geometry>
     </visual>
+    <inertial>
+      <mass value="1e-5" />
+      <origin xyz="0 0 0" rpy="0 0 0"/>
+      <inertia ixx="1e-6" ixy="0" ixz="0" iyy="1e-6" iyz="0" izz="1e-6" />
+    </inertial>
   </link>
   <link name="base_link">
